File: TMotor_Rev0.sch (EAGLE design)
At the start: 33 parts, among them U1 INA125U, U2 INA125U

Commit message: Pre check completion, with pogo pins
Parts:
- removed BRKOUT: (no value), SparkFun-Connectors:CONN_03X2SHROUD
- removed D2: 1N4004, diode:1N4004
- added J1, J2: (no value), SparkFun-Connectors:CONN_10"
- added J3: (no value), SparkFun-Connectors:CONN_07
- added POGO: (no value), pinhead:PINHD-2X3
- added SWD: 20317, microbuilder:JTAG-CORTEXBOXPOSTS
- added U$9: XT30, Ben_Library:XT30
Connections:
- net MD_VCC renamed L7_VIN
- net N$2 renamed PF_VCC
- removed net 5V: C3.2, C5.1, D2.A, INA219.VS, L7805.OUTPUT
- removed net D11: USB.D11
- removed net D12: USB.D12
- removed net D8: USB.D8
- removed net D9: USB.D9
- removed net N$1: FUSE.2
- removed net PWM-RL: USB.D10
- new net CAN_CS: J1.2, USB.D10
- new net CAN_INT: J1.6, USB.D8
- new net H_CS: J2.9, J3.3
- new net H_INT: J2.5, J3.7
- new net H_MISO: J2.8, J3.4
- new net H_MOSI: J2.7, J3.5
- new net H_SCK: J2.6, J3.6
- new net LLS_OE: J1.10, USB.D9
- new net MISO: J1.3, USB.D12
- new net MOSI: J1.4, USB.D11
- new net N$27: J1.7
- new net N$28: J1.8
- new net N$29: J1.9
- new net NRESET: POGO.5, SWD.NRESET
- new net SCK: J1.5, USB.D13
- new net SW3.3V: POGO.2, SWD.VCC
- new net SWCLK: POGO.4, SWD.SWDCLK
- new net SWDIO: POGO.1, SWD.SWDIO
- new net SWGND: POGO.6, SWD.GND@1, SWD.GND@2
- new net VCC: FUSE.2, U$9.+
- net 3.3V: now also J1.1; no longer BRKOUT.2, BRKOUT.4, BRKOUT.6
- net A2: no longer BRKOUT.1
- net A3: no longer BRKOUT.5
- net GND: now also J2.1, J3.2, U$9.-
- net VIN: now also C3.2, C5.1, INA219.VS, J2.10, J3.1, L7805.OUTPUT; no longer D2.C

Commit message: Final V0 sent to oshpark
Parts:
- R14: value 3.3k -> 470R
- R16: value 1k -> 470R
Changed lines of the file:
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@@
 <part name="TRQ-RA" library="SparkFun-Connectors" library_urn="urn:adsk.eagle:library:513" deviceset="CONN_03X2" device="SHROUD" package3d_urn="urn:adsk.eagle:package:38264/1"/>
 <part name="GND14" library="SparkFun-PowerSymbols" library_urn="urn:adsk.eagle:library:530" deviceset="GND" device=""/>
-<part name="R14" library="rcl" library_urn="urn:adsk.eagle:library:334" deviceset="R-US_" device="0207/10" package3d_urn="urn:adsk.eagle:package:23491/1" value="3.3k"/>
+<part name="R14" library="rcl" library_urn="urn:adsk.eagle:library:334" deviceset="R-US_" device="0207/10" package3d_urn="urn:adsk.eagle:package:23491/1" value="470R"/>
 <part name="C6" library="rcl" library_urn="urn:adsk.eagle:library:334" deviceset="C-EU" device="050-024X044" package3d_urn="urn:adsk.eagle:package:23643/1" value="100nF"/>
 <part name="C7" library="rcl" library_urn="urn:adsk.eagle:library:334" deviceset="C-EU" device="050-024X044" package3d_urn="urn:adsk.eagle:package:23643/1" value="100nF"/>
@@
 <part name="TRQ-LA" library="SparkFun-Connectors" library_urn="urn:adsk.eagle:library:513" deviceset="CONN_03X2" device="SHROUD" package3d_urn="urn:adsk.eagle:package:38264/1"/>
 <part name="GND18" library="SparkFun-PowerSymbols" library_urn="urn:adsk.eagle:library:530" deviceset="GND" device=""/>
-<part name="R16" library="rcl" library_urn="urn:adsk.eagle:library:334" deviceset="R-US_" device="0207/10" package3d_urn="urn:adsk.eagle:package:23491/1" value="1k"/>
+<part name="R16" library="rcl" library_urn="urn:adsk.eagle:library:334" deviceset="R-US_" device="0207/10" package3d_urn="urn:adsk.eagle:package:23491/1" value="470R"/>
 <part name="C12" library="rcl" library_urn="urn:adsk.eagle:library:334" deviceset="C-EU" device="050-024X044" package3d_urn="urn:adsk.eagle:package:23643/1" value="100nF"/>
 <part name="C13" library="rcl" library_urn="urn:adsk.eagle:library:334" deviceset="C-EU" device="050-024X044" package3d_urn="urn:adsk.eagle:package:23643/1" value="100nF"/>

Commit message: First Rev1 changes
Parts:
- removed FAN: (no value), SparkFun-Connectors:CONN_02
- removed POGO: (no value), pinhead:PINHD-2X3
- removed SWD: 20317, microbuilder:JTAG-CORTEXBOXPOSTS
Connections:
- removed net NRESET: POGO.5, SWD.NRESET
- removed net SW3.3V: POGO.2, SWD.VCC
- removed net SWCLK: POGO.4, SWD.SWDCLK
- removed net SWDIO: POGO.1, SWD.SWDIO
- removed net SWGND: POGO.6, SWD.GND@1, SWD.GND@2
- net GND: no longer FAN.2
- net VIN: no longer FAN.1
Changed lines of the file:
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@@
 <part name="D1" library="diode" library_urn="urn:adsk.eagle:library:210" deviceset="1N5400" device="" package3d_urn="urn:adsk.eagle:package:43365/2"/>
 <part name="GND7" library="SparkFun-PowerSymbols" library_urn="urn:adsk.eagle:library:530" deviceset="GND" device=""/>
-<part name="FAN" library="SparkFun-Connectors" library_urn="urn:adsk.eagle:library:513" deviceset="CONN_02" device="" package3d_urn="urn:adsk.eagle:package:38039/1"/>
-<part name="GND16" library="SparkFun-PowerSymbols" library_urn="urn:adsk.eagle:library:530" deviceset="GND" device=""/>
 <part name="C9" library="rcl" library_urn="urn:adsk.eagle:library:334" deviceset="C-EU" device="050-024X044" package3d_urn="urn:adsk.eagle:package:23643/1" value="0.1uF"/>
 <part name="R1" library="rcl" library_urn="urn:adsk.eagle:library:334" deviceset="R-US_" device="0207/10" package3d_urn="urn:adsk.eagle:package:23491/1" value="10R"/>
@@
 <part name="GND4" library="SparkFun-PowerSymbols" library_urn="urn:adsk.eagle:library:530" deviceset="GND" device=""/>
 <part name="GND5" library="SparkFun-PowerSymbols" library_urn="urn:adsk.eagle:library:530" deviceset="GND" device=""/>
-<part name="SWD" library="microbuilder" deviceset="JTAG-CORTEX" device="BOXPOSTS" value="20317"/>
-<part name="POGO" library="pinhead" library_urn="urn:adsk.eagle:library:325" deviceset="PINHD-2X3" device="" package3d_urn="urn:adsk.eagle:package:22462/2"/>
 <part name="U$9" library="Ben_Library" deviceset="XT30" device=""/>
 </parts>
@@
 <attribute name="VALUE" x="-167.8686" y="165.1" size="1.778" layer="96" rot="R90"/>
 </instance>
-<instance part="FAN" gate="G$1" x="-294.64" y="190.5" smashed="yes" rot="R180">
-<attribute name="VALUE" x="-292.1" y="195.326" size="1.778" layer="96" font="vector" rot="R180"/>
-<attribute name="NAME" x="-292.1" y="184.912" size="1.778" layer="95" font="vector" rot="R180"/>
-</instance>
-<instance part="GND16" gate="1" x="-309.88" y="177.8" smashed="yes" rot="MR0">
-<attribute name="VALUE" x="-309.88" y="177.546" size="1.778" layer="96" rot="MR0" align="top-center"/>
-</instance>
 <instance part="C9" gate="G$1" x="-175.26" y="218.44" smashed="yes" rot="MR0">
 <attribute name="NAME" x="-176.784" y="218.821" size="1.778" layer="95" rot="MR0"/>
@@
 <instance part="GND5" gate="1" x="-68.58" y="200.66" smashed="yes" rot="MR0">
 <attribute name="VALUE" x="-68.58" y="200.406" size="1.778" layer="96" rot="MR0" align="top-center"/>
-</instance>
-<instance part="SWD" gate="G$1" x="-114.3" y="109.22" smashed="yes">
-<attribute name="NAME" x="-120.65" y="117.475" size="1.27" layer="95"/>
-<attribute name="VALUE" x="-120.65" y="99.695" size="1.27" layer="96"/>
-</instance>
-<instance part="POGO" gate="A" x="-162.56" y="109.22" smashed="yes" rot="R180">
-<attribute name="NAME" x="-156.21" y="103.505" size="1.778" layer="95" rot="R180"/>
-<attribute name="VALUE" x="-156.21" y="116.84" size="1.778" layer="96" rot="R180"/>
 </instance>
 <instance part="U$9" gate="G$1" x="-71.12" y="220.98" smashed="yes" rot="R90"/>
@@
 </segment>
 <segment>
-<pinref part="FAN" gate="G$1" pin="2"/>
-<wire x1="-302.26" y1="187.96" x2="-309.88" y2="187.96" width="0.1524" layer="91"/>
-<wire x1="-309.88" y1="187.96" x2="-309.88" y2="180.34" width="0.1524" layer="91"/>
-<pinref part="GND16" gate="1" pin="GND"/>
-</segment>
-<segment>
 <pinref part="INA219" gate="A" pin="A1"/>
 <wire x1="-243.84" y1="213.36" x2="-248.92" y2="213.36" width="0.1524" layer="91"/>
@@
 </net>
 <net name="VIN" class="0">
-<segment>
-<pinref part="FAN" gate="G$1" pin="1"/>
-<label x="-314.96" y="193.04" size="1.778" layer="95"/>
-<wire x1="-302.26" y1="190.5" x2="-312.42" y2="190.5" width="0.1524" layer="91"/>
-<junction x="-312.42" y="190.5"/>
-</segment>
 <segment>
 <wire x1="-91.44" y1="195.58" x2="-180.34" y2="195.58" width="0.1524" layer="91"/>
@@
 </segment>
 </net>
-<net name="SWCLK" class="0">
-<segment>
-<pinref part="POGO" gate="A" pin="4"/>
-<wire x1="-167.64" y1="109.22" x2="-175.26" y2="109.22" width="0.1524" layer="91"/>
-<label x="-182.88" y="109.22" size="1.778" layer="95"/>
-</segment>
-<segment>
-<pinref part="SWD" gate="G$1" pin="SWDCLK"/>
-<wire x1="-106.68" y1="111.76" x2="-101.6" y2="111.76" width="0.1524" layer="91"/>
-<label x="-106.68" y="111.76" size="1.778" layer="95"/>
-</segment>
-</net>
-<net name="SWGND" class="0">
-<segment>
-<pinref part="POGO" gate="A" pin="6"/>
-<wire x1="-167.64" y1="111.76" x2="-175.26" y2="111.76" width="0.1524" layer="91"/>
-<label x="-182.88" y="111.76" size="1.778" layer="95"/>
-</segment>
-<segment>
-<pinref part="SWD" gate="G$1" pin="GND@1"/>
-<pinref part="SWD" gate="G$1" pin="GND@2"/>
-<wire x1="-121.92" y1="111.76" x2="-121.92" y2="109.22" width="0.1524" layer="91"/>
-<wire x1="-121.92" y1="111.76" x2="-129.54" y2="111.76" width="0.1524" layer="91"/>
-<junction x="-121.92" y="111.76"/>
-<label x="-132.08" y="111.76" size="1.778" layer="95"/>
-</segment>
-</net>
-<net name="SW3.3V" class="0">
-<segment>
-<pinref part="POGO" gate="A" pin="2"/>
-<wire x1="-167.64" y1="106.68" x2="-175.26" y2="106.68" width="0.1524" layer="91"/>
-<label x="-182.88" y="106.68" size="1.778" layer="95"/>
-</segment>
-<segment>
-<pinref part="SWD" gate="G$1" pin="VCC"/>
-<wire x1="-121.92" y1="114.3" x2="-129.54" y2="114.3" width="0.1524" layer="91"/>
-<label x="-132.08" y="114.3" size="1.778" layer="95"/>
-</segment>
-</net>
-<net name="NRESET" class="0">
-<segment>
-<pinref part="POGO" gate="A" pin="5"/>
-<wire x1="-160.02" y1="111.76" x2="-154.94" y2="111.76" width="0.1524" layer="91"/>
-<label x="-154.94" y="111.76" size="1.778" layer="95"/>
-</segment>
-<segment>
-<pinref part="SWD" gate="G$1" pin="NRESET"/>
-<wire x1="-106.68" y1="104.14" x2="-101.6" y2="104.14" width="0.1524" layer="91"/>
-<label x="-106.68" y="104.14" size="1.778" layer="95"/>
-</segment>
-</net>
-<net name="SWDIO" class="0">
-<segment>
-<pinref part="POGO" gate="A" pin="1"/>
-<wire x1="-160.02" y1="106.68" x2="-154.94" y2="106.68" width="0.1524" layer="91"/>
-<label x="-154.94" y="106.68" size="1.778" layer="95"/>
-</segment>
-<segment>
-<pinref part="SWD" gate="G$1" pin="SWDIO"/>
-<wire x1="-106.68" y1="114.3" x2="-101.6" y2="114.3" width="0.1524" layer="91"/>
-<label x="-106.68" y="114.3" size="1.778" layer="95"/>
-</segment>
-</net>

Commit message: Rev1 Final chance
Parts:
- removed C5, C9: 0.1uF, rcl:C-EU050-024X044
- removed INA219: (no value), INA219:INA219AIDR
- removed R1, R2: 10R, rcl:R-US_0207/10
- removed SHUNT: 2mOhm, ShuntResistor:CSNL2512FT2L00
- added C1: 1mF, rcl:CPOL-USE5-10.5
Connections:
- removed net N$23: C9.1, INA219.VIN+, R2.1
- removed net N$26: C9.2, INA219.VIN-, R1.1
- removed net PF_VCC: FUSE.1, R2.2, SHUNT.2
- net GND: now also C1.-; no longer C5.2, INA219.A0, INA219.A1, INA219.GND
- net L7_VIN: now also FUSE.1; no longer R1.2, SHUNT.1
- net SCL1: no longer INA219.SCL
- net SDA1: no longer INA219.SDA
- net VCC: now also C1.+
- net VIN: no longer C5.1, INA219.VS
