File: TMotor_Rev0.brd (EAGLE design)
At the start: 56.5 x 66.3 mm, 37 parts, among them U1 INA125U, U2 INA125U

Commit message: First Rev1 changes
Parts:
- removed FAN: (no value), SparkFun-Connectors:1X02
- removed POGO: (no value), pinhead:2X03
- removed SWD: 20317, microbuilder:2X05_1.27MM_BOX_POSTS
- moved C7 33.0 mm to (52.1, 8.26), turned to 0 degrees
- moved C15 27.5 mm to (47.6, 40.0), turned to 0 degrees
- moved C13 25.5 mm to (15.6, 7.62), turned to 0 degrees
- moved C8 24.1 mm to (51.1, 13.3), flipped to the bottom, turned to 90 degrees
- moved R14 22.7 mm to (43.8, 14.9), turned to 180 degrees
- moved U2 20.3 mm to (43.5, 9.84), turned to 90 degrees
- moved C14 19.7 mm to (14.9, 12.4), turned to 90 degrees
- moved U1 17.8 mm to (7.30, 9.53), turned to 90 degrees
- moved R16 14.0 mm to (7.94, 14.6), turned to 180 degrees
- moved TRQ-RA 12.2 mm to (47.6, 1.59)
- moved TRQ-LA 12.1 mm to (8.26, 1.27)
- moved C12 10.2 mm to (12.7, 24.8), turned to 90 degrees
- moved C6 8.55 mm to (27.9, 24.8), turned to 90 degrees
- moved R7 2.93 mm to (25.4, 14.0)
- moved R8 2.88 mm to (22.9, 16.5)
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Connections:
- removed net NRESET: POGO.5, SWD.10
- removed net SW3.3V: POGO.2, SWD.1
- removed net SWCLK: POGO.4, SWD.4
- removed net SWDIO: POGO.1, SWD.2
- removed net SWGND: POGO.6, SWD.3, SWD.5
- net GND: no longer FAN.2
- net VIN: no longer FAN.1
Routing:
- net N$9: track 33.0 -> 9.81 mm, vias 1 -> 0
- net N$8: track 29.1 -> 13.2 mm, vias 2 -> 0
- net SW3.3V: track 14.3 -> 0.00 mm
- net SWGND: track 13.9 -> 0.00 mm, vias 1 -> 0
- net A6: track 12.0 -> 24.6 mm
- net VIN: track 101.6 -> 92.4 mm
- net N$11: track 19.9 -> 10.7 mm, vias 1 -> 0
- net N$7: track 2.24 -> 11.4 mm, vias 0 -> 2
- net 3.3V: track 99.6 -> 108.2 mm
- net GND: track 15.6 -> 7.51 mm, vias 2 -> 0
- net SWCLK: track 7.98 -> 0.00 mm
- net N$6: track 5.41 -> 12.8 mm, vias 0 -> 2
- net N$10: track 20.9 -> 14.1 mm, vias 2 -> 0
- net N$12: track 4.41 -> 11.0 mm, vias 0 -> 2
- net A2: track 18.5 -> 25.1 mm
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Other:
- board size 56.5 x 66.3 mm -> 56.5 x 79 mm

Commit message: Rev1 Final chance
Parts:
- removed C5, C9: 0.1uF, rcl:C050-024X044
- removed INA219: (no value), INA219:D8_TEX
- removed R1, R2: 10R, rcl:0207/10
- removed SHUNT: 2mOhm, ShuntResistor:STA_CSNL2512(2)_STP
- added C1: 1mF, rcl:E5-10,5
- moved C16 20.2 mm to (36.8, 45.4), turned to 270 degrees
- moved D1 18.1 mm to (46.4, 63.5)
- moved C15 16.8 mm to (43.2, 23.8)
- moved FUSE 10.4 mm to (29.2, 52.4), turned to 90 degrees
- moved C3 9.84 mm to (47.9, 42.5), turned to 180 degrees
- moved C4 1.00 mm to (48.6, 52.4)
- moved C14 0.95 mm to (15.9, 12.4)
- moved R14 0.95 mm to (43.8, 15.9)
- moved U2 0.95 mm to (42.5, 9.84)
- moved C13 0.63 mm to (16.2, 7.62)
- moved C7 0.32 mm to (51.8, 8.26)
- moved C8 0.32 mm to (51.4, 13.3)
- moved C12 0.32 mm to (12.7, 25.1)
- moved C19 0.32 mm to (17.8, 25.1)
- moved C20 0.32 mm to (20.3, 25.1)
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Connections:
- removed net N$23: C9.1, INA219.8, R2.1
- removed net N$26: C9.2, INA219.7, R1.1
- removed net PF_VCC: FUSE.1, R2.2, SHUNT.2
- net GND: now also C1.-; no longer C5.2, INA219.1, INA219.2, INA219.6
- net L7_VIN: now also FUSE.1; no longer R1.2, SHUNT.1
- net SCL1: no longer INA219.4
- net SDA1: no longer INA219.3
- net VCC: now also C1.+
- net VIN: no longer C5.1, INA219.5
Routing:
- net SDA1: track 31.2 -> 0.00 mm
- net SCL1: track 30.2 -> 0.00 mm
- net L7_VIN: track 35.4 -> 23.4 mm
- net VIN: track 92.4 -> 80.8 mm
- net PF_VCC: track 8.88 -> 0.00 mm
- net N$23: track 8.70 -> 0.00 mm
- net VCC: track 4.14 -> 12.1 mm
- net N$26: track 4.26 -> 0.00 mm
- net CAN_CS: track 10.3 -> 12.4 mm, vias 0 -> 2
- net N$6: track 12.8 -> 14.7 mm
- net SCK: track 25.2 -> 27.1 mm, vias 0 -> 2
- net N$9: track 9.81 -> 11.1 mm
- net N$10: track 14.1 -> 15.0 mm
- net N$8: track 13.2 -> 14.1 mm
- net GND: track 7.51 -> 8.31 mm, vias 0 -> 29
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- added copper zone on layer 16, net GND
- removed copper zone on layer 1, net GND

Commit message: Incremented Version number
Routing:
- net VIN: track 80.8 -> 80.3 mm
Other:
- board text added: "AK_Board V1"
- board text removed: "AK_Board V0"
Changed lines of the file:
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@@
 <circle x="52" y="70" radius="1.75" width="0.254" layer="20"/>
 <circle x="52" y="22" radius="1.75" width="0.254" layer="20"/>
-<text x="8.255" y="70.1675" size="1.778" layer="21">AK_Board V0</text>
+<text x="8.255" y="70.1675" size="1.778" layer="21">AK_Board V1</text>
 <text x="1.5875" y="62.5475" size="1.778" layer="21">CAN</text>
 <text x="1.5875" y="56.8325" size="1.778" layer="21">LLS</text>
@@
 <wire x1="45.2988" y1="45.4025" x2="45.3263" y2="45.375" width="0.4064" layer="1"/>
 <wire x1="12.065" y1="45.4025" x2="45.2988" y2="45.4025" width="0.4064" layer="1"/>
-<wire x1="45.3263" y1="44.8437" x2="45.3263" y2="45.375" width="0.4064" layer="1"/>
-<wire x1="45.3263" y1="45.375" x2="45.3263" y2="42.6212" width="0.4064" layer="1"/>
-<wire x1="45.3263" y1="42.6212" x2="45.4025" y2="42.545" width="0.4064" layer="1"/>
 <wire x1="45.4025" y1="42.545" x2="45.4025" y2="28.575" width="0.4064" layer="1"/>
 <wire x1="45.4025" y1="28.575" x2="40.64" y2="23.8125" width="0.4064" layer="1"/>
+<wire x1="45.3263" y1="45.375" x2="45.4025" y2="45.2988" width="0.4064" layer="1"/>
+<wire x1="45.4025" y1="45.2988" x2="45.4025" y2="42.545" width="0.4064" layer="1"/>
 </signal>
 <signal name="3.3V">
