File: TMotor_Rev0_5.sch (EAGLE design)
At the start: 79 parts, among them U1 INA125U, U10 DEV-16771, U2 INA125U, U3 INA125U, U4 INA125U, U5 SN65HVD230MDREP

Commit message: Comments added.
Other:
- note added: "External power supply"
- note added: "Here is to measure the voltage. INA219 is a sensor that will use the info captured from pins VIN+ and VIN- to estimate the voltage magnitude of the power supply. Note that eventually both VIN+ and VIN- are indirectly connected to the positive terminals of the battery voltages measured. INA219 requires an external SHUNT circuit as shown here."
- note added: "VS: Power supply for the INA 219 sensor (INA 219 takes 3 to 5.5 V) GND: Ground for the INA 219 sensor"
- note added: "Verify: CANTX is the CAN BUS transmission pin Verify: CANRX is the CAN BUS receiver pin"
Changed lines of the file:
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@@
 <description>Motor Drivers &amp; Power</description>
 <plain>
+<text x="-91.44" y="292.1" size="1.778" layer="91">External power supply</text>
+<text x="-50.8" y="330.2" size="1.778" layer="91">External power supply</text>
+<text x="-10.16" y="330.2" size="1.778" layer="91">External power supply</text>
+<text x="35.56" y="330.2" size="1.778" layer="91">External power supply</text>
+<text x="78.74" y="330.2" size="1.778" layer="91">External power supply</text>
+<text x="-208.28" y="226.06" size="1.778" layer="91">Here is to measure the voltage.
+INA219 is a sensor that will use the info captured from pins VIN+ and VIN- to estimate the voltage magnitude of the power supply.
+Note that eventually both VIN+ and VIN- are indirectly connected to the positive terminals of the battery voltages measured.
+INA219 requires an external SHUNT circuit as shown here.</text>
+<text x="-238.76" y="190.5" size="1.778" layer="91">VS: Power supply for the INA 219 sensor (INA 219 takes 3 to 5.5 V)
+GND: Ground for the INA 219 sensor</text>
+<text x="-317.5" y="106.68" size="1.778" layer="91">Verify: CANTX is the CAN BUS  transmission pin
+Verify: CANRX is the CAN BUS receiver pin</text>
 </plain>
 <instances>
@@
 </drawing>
 <compatibility>
+<note version="6.3" minversion="6.2.2" severity="warning">
+Since Version 6.2.2 text objects can contain more than one line,
+which will not be processed correctly with this version.
+</note>
 <note version="8.2" severity="warning">
 Since Version 8.2, EAGLE supports online libraries. The ids
